File: Base/KiCAD/BarePi_Base.kicad_pcb (KiCad board)
At the start: 2 copper layers, 65 x 42 mm, 28 parts, among them IC1 HT7533-1, J1 IN, J2 OUT, J3 AudioJack, J4 POWER, J5 Micro SD Card, J6 3V3 Stabilizer, SW1 RESET

Commit message: init
Connections:
- J2 pad 17: /PWM_L -> unconnected-(J2-Pin_17-Pad17)
- J2 pad 18: /PWM_R -> unconnected-(J2-Pin_18-Pad18)
Routing:
- net /PWM_L: track 38.9 -> 7.51 mm
- net /PWM_R: track 36.1 -> 11.8 mm
Changed lines of the file:
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@@
 	(net 49 "Net-(D2-A)")
 	(net 50 "/USR_LED")
+	(net 51 "unconnected-(J2-Pin_17-Pad17)")
+	(net 52 "unconnected-(J2-Pin_18-Pad18)")
 	(footprint "Raspberry:Raspberry_OUT_PinSocket_2x20_P2.54mm_Horizontal"
 		(locked yes)
@@
 			(layers "*.Cu" "*.Mask")
 			(remove_unused_layers no)
-			(net 5 "/PWM_L")
+			(net 51 "unconnected-(J2-Pin_17-Pad17)")
 			(pinfunction "Pin_17")
-			(pintype "passive")
+			(pintype "passive+no_connect")
 			(thermal_bridge_angle 45)
 		)
@@
 			(layers "*.Cu" "*.Mask")
 			(remove_unused_layers no)
-			(net 28 "/PWM_R")
+			(net 52 "unconnected-(J2-Pin_18-Pad18)")
 			(pinfunction "Pin_18")
-			(pintype "passive")
+			(pintype "passive+no_connect")
 			(thermal_bridge_angle 45)
 		)
@@
 	)
 	(segment
-		(start 29.989 27.95095)
-		(end 29.964 27.97595)
-		(width 0.33)
-		(layer "B.Cu")
-		(net 5)
-	)
-	(segment
-		(start 28.69 4.23)
-		(end 29.989 5.529)
-		(width 0.4)
-		(layer "B.Cu")
-		(net 5)
-	)
-	(segment
-		(start 29.989 31.721)
-		(end 28.69 33.02)
-		(width 0.4)
-		(layer "B.Cu")
-		(net 5)
-	)
-	(segment
-		(start 29.964 31.696)
-		(end 29.989 31.721)
-		(width 0.33)
-		(layer "B.Cu")
-		(net 5)
-	)
-	(segment
-		(start 31.825 11.81005)
-		(end 31.825 26.11495)
-		(width 0.4)
-		(layer "B.Cu")
-		(net 5)
-	)
-	(segment
-		(start 29.956 8.467465)
-		(end 29.989 8.500465)
-		(width 0.33)
-		(layer "B.Cu")
-		(net 5)
-	)
-	(segment
-		(start 31.825 26.11495)
-		(end 29.989 27.95095)
-		(width 0.4)
-		(layer "B.Cu")
-		(net 5)
-	)
-	(segment
-		(start 29.989 8.500465)
-		(end 31.625 10.136466)
-		(width 0.4)
-		(layer "B.Cu")
-		(net 5)
-	)
-	(segment
-		(start 31.625 11.61005)
-		(end 31.825 11.81005)
-		(width 0.4)
-		(layer "B.Cu")
-		(net 5)
-	)
-	(segment
-		(start 29.964 27.97595)
-		(end 29.964 31.696)
-		(width 0.33)
-		(layer "B.Cu")
-		(net 5)
-	)
-	(segment
-		(start 29.989 5.529)
-		(end 29.956 5.562)
-		(width 0.33)
-		(layer "B.Cu")
-		(net 5)
-	)
-	(segment
-		(start 31.625 10.136466)
-		(end 31.625 11.61005)
-		(width 0.4)
-		(layer "B.Cu")
-		(net 5)
-	)
-	(segment
-		(start 29.956 5.562)
-		(end 29.956 8.467465)
-		(width 0.33)
-		(layer "B.Cu")
-		(net 5)
-	)
-	(segment
 		(start 22.15 9.911916)
 		(end 22.15 9.916158)
@@
 	)
 	(segment
-		(start 30.891 10.392415)
-		(end 28.69 8.191415)
-		(width 0.4)
-		(layer "B.Cu")
-		(net 28)
-	)
-	(segment
-		(start 28.69 30.48)
-		(end 28.69 28.26)
-		(width 0.4)
-		(layer "B.Cu")
-		(net 28)
-	)
-	(segment
-		(start 31.124 19.124)
-		(end 31.124 25.824586)
-		(width 0.4)
-		(layer "B.Cu")
-		(net 28)
-	)
-	(segment
 		(start 28.69 8.191415)
 		(end 28.69 6.77)
 		(width 0.4)
 		(layer "B.Cu")
-		(net 28)
-	)
-	(segment
-		(start 31.124 25.824586)
-		(end 30.891 26.057586)
-		(width 0.4)
-		(layer "B.Cu")
-		(net 28)
-	)
-	(segment
-		(start 30.891 26.057586)
-		(end 30.891 26.059)
-		(width 0.4)
-		(layer "B.Cu")
-		(net 28)
-	)
-	(segment
-		(start 28.69 28.26)
-		(end 30.891 26.059)
-		(width 0.4)
-		(layer "B.Cu")
-		(net 28)
-	)
-	(segment
-		(start 30.891 18.891)
-		(end 31.124 19.124)
-		(width 0.4)
-		(layer "B.Cu")
-		(net 28)
-	)
-	(segment
-		(start 30.891 10.392415)
-		(end 30.891 18.891)
-		(width 0.4)
-		(layer "B.Cu")
