File: Base/KiCAD/BarePi_Base.kicad_sch (KiCad schematic)
At the start: 24 parts, among them IC1 HT7533-1, J1 IN, J2 OUT, J3 AudioJack, J4 POWER, J5 Micro SD Card, J6 3V3 Stabilizer, SW1 RESET

Commit message: init
Connections:
- net PWM_L: no longer J2.17 (Pin_17)
- net PWM_R: no longer J2.18 (Pin_18)
- no-connect marks 5 -> 7
Changed lines of the file:
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@@
+	)
+	(no_connect
+		(at 210.82 83.82)
 	)
 	(no_connect
@@
 	)
 	(no_connect
+		(at 175.26 83.82)
+	)
+	(no_connect
 		(at 132.08 124.46)
 	)
@@
 	(wire
 		(pts
-			(xy 162.56 83.82) (xy 175.26 83.82)
-		)
-		(stroke
-			(width 0)
-			(type default)
-		)
-	)
-	(wire
-		(pts
 			(xy 162.56 81.28) (xy 175.26 81.28)
 		)
@@
 		(pts
 			(xy 210.82 139.7) (xy 215.9 139.7)
-		)
-		(stroke
-			(width 0)
-			(type default)
-		)
-	)
-	(wire
-		(pts
-			(xy 210.82 83.82) (xy 223.52 83.82)
 		)
 		(stroke
@@
 		)
 	)
-	(label "PWM_R"
-		(at 223.52 83.82 180)
-		(effects
-			(font
-				(size 1.27 1.27)
-			)
-			(justify right bottom)
-		)
-	)
 	(label "LCD_MOSI"
 		(at 162.56 93.98 0)
@@
 		)
 	)
-	(label "PWM_L"
-		(at 162.56 83.82 0)
-		(effects
-			(font
-				(size 1.27 1.27)
-			)
-			(justify left bottom)
-		)
-	)
