File: BusExp/KiCAD/BarePi_BusExp.kicad_sch (KiCad schematic)
At the start: 4 parts, among them J1 IN, J2 OUT, J3 IN, J4 OUT

Commit message: init
Connections:
- net 3V3 renamed 3V3_1
- net 3V3_1: no longer J1.4 (Pin_4), J2.4 (Pin_4), J3.4 (Pin_4), J4.4 (Pin_4)
- net 5V renamed 5V_1
- net 5V_1: no longer J1.2 (Pin_2), J2.2 (Pin_2), J3.2 (Pin_2), J4.2 (Pin_2)
- net GND renamed GND_1
- net GND_1: no longer J1.40 (Pin_40), J2.40 (Pin_40), J3.40 (Pin_40), J4.40 (Pin_40)
- new net 3V3_2: J1.4 (Pin_4), J2.4 (Pin_4), J3.4 (Pin_4), J4.4 (Pin_4)
- new net 5V_2: J1.2 (Pin_2), J2.2 (Pin_2), J3.2 (Pin_2), J4.2 (Pin_2)
- new net GND_2: J1.40 (Pin_40), J2.40 (Pin_40), J3.40 (Pin_40), J4.40 (Pin_40)
Changed lines of the file:
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@@
 		)
 	)
-	(label "5V"
+	(label "5V_1"
 		(at 149.86 58.42 0)
 		(effects
@@
 		)
 	)
-	(label "GND"
+	(label "GND_1"
 		(at 83.82 106.68 0)
 		(effects
@@
 		)
 	)
-	(label "GND"
+	(label "GND_1"
 		(at 149.86 162.56 0)
 		(effects
@@
 		)
 	)
-	(label "GND"
+	(label "GND_2"
 		(at 210.82 106.68 180)
 		(effects
@@
 		)
 	)
-	(label "5V"
+	(label "5V_2"
 		(at 144.78 58.42 180)
 		(effects
@@
 		)
 	)
-	(label "3V3"
+	(label "3V3_2"
 		(at 210.82 60.96 180)
 		(effects
@@
 		)
 	)
-	(label "GND"
+	(label "GND_1"
 		(at 149.86 106.68 0)
 		(effects
@@
 		)
 	)
-	(label "5V"
+	(label "5V_1"
 		(at 149.86 114.3 0)
 		(effects
@@
 		)
 	)
-	(label "3V3"
+	(label "3V3_2"
 		(at 210.82 116.84 180)
 		(effects
@@
 		)
 	)
-	(label "GND"
+	(label "GND_1"
 		(at 83.82 162.56 0)
 		(effects
@@
 		)
 	)
-	(label "GND"
+	(label "GND_2"
 		(at 210.82 162.56 180)
 		(effects
@@
 		)
 	)
-	(label "5V"
+	(label "5V_2"
 		(at 210.82 114.3 180)
 		(effects
@@
 		)
 	)
-	(label "3V3"
+	(label "3V3_2"
 		(at 144.78 116.84 180)
 		(effects
@@
 		)
 	)
-	(label "3V3"
+	(label "3V3_2"
 		(at 144.78 60.96 180)
 		(effects
@@
 		)
 	)
-	(label "GND"
+	(label "GND_2"
 		(at 144.78 106.68 180)
 		(effects
@@
 		)
 	)
-	(label "5V"
+	(label "5V_2"
 		(at 144.78 114.3 180)
 		(effects
@@
 		)
 	)
-	(label "GND"
+	(label "GND_2"
 		(at 144.78 162.56 180)
 		(effects
@@
 		)
 	)
-	(label "3V3"
+	(label "3V3_1"
 		(at 149.86 116.84 0)
 		(effects
@@
 		)
 	)
-	(label "5V"
+	(label "5V_1"
 		(at 83.82 58.42 0)
 		(effects
@@
 		)
 	)
-	(label "3V3"
+	(label "3V3_1"
 		(at 83.82 60.96 0)
 		(effects
@@
 		)
 	)
-	(label "5V"
+	(label "5V_2"
 		(at 210.82 58.42 180)
 		(effects
@@
 		)
 	)
-	(label "3V3"
+	(label "3V3_1"
 		(at 83.82 116.84 0)
 		(effects
@@
 		)
 	)
-	(label "5V"
+	(label "5V_1"
 		(at 83.82 114.3 0)
 		(effects
@@
 		)
 	)
-	(label "3V3"
+	(label "3V3_1"
 		(at 149.86 60.96 0)
 		(effects
