File: CalcKey/KiCAD/BarePi_CalcKey.kicad_pcb (KiCad board)
At the start: 2 copper layers, 65 x 106 mm, 55 parts, among them J1 IN, J2 OUT, J3 WCH-LINK, U1 CH32V002F4P6

Commit message: init
Parts:
- added R1: 15K, Resistor_SMD:R_1206_3216Metric_Pad1.30x1.75mm_HandSolder, F.Cu at (21.6, 11.9)
- added R2: 15K, Resistor_SMD:R_1206_3216Metric_Pad1.30x1.75mm_HandSolder, F.Cu at (25.0, 11.9)
- moved JP1 1.39 mm to (61.0, 9.38), turned to 0 degrees
Routing:
- net /BUS_SCL: track 122.6 -> 126.3 mm
- net /BUS_SDA: track 118.5 -> 120.6 mm
- net /ROW2: track 117.3 -> 118.6 mm
- net /3V3: track 148.4 -> 149.0 mm
