File: LCD160x80/KiCAD/BarePi_LCD160x80.kicad_pcb (KiCad board)
At the start: 2 copper layers, 65 x 49 mm, 16 parts, among them J1 IN, J2 OUT, J3 LCD, J4 WCH-LINK, U1 CH32V002J4M6

Commit message: init
Parts:
- added R2: 15K, Resistor_SMD:R_1206_3216Metric_Pad1.30x1.75mm_HandSolder, F.Cu at (14.4, 22.0)
- added R3: 15K, Resistor_SMD:R_1206_3216Metric_Pad1.30x1.75mm_HandSolder, B.Cu at (12.0, 15.6)
- R1: value 10K -> 15K
Routing:
- net /3V3: track 114.6 -> 117.3 mm
- net /BUS_SDA: track 84.2 -> 85.9 mm
