File: LCD16x2/KiCAD/BarePi_LCD16x2.kicad_pcb (KiCad board)
At the start: 2 copper layers, 80 x 61 mm, 21 parts, among them J1 IN, J2 OUT, J3 Backlight, J4 WCH-LINK, SW1 VO_DN, SW2 VO_UP, U1 CH32V002A4M6, U2 DM1602A

Commit message: init
Parts:
- added R2: 15K, Resistor_SMD:R_1206_3216Metric_Pad1.30x1.75mm_HandSolder, F.Cu at (16.8, 26.3)
- added R3: 15K, Resistor_SMD:R_1206_3216Metric_Pad1.30x1.75mm_HandSolder, F.Cu at (16.8, 23.1)
- moved C1 1.05 mm to (55.5, 26.3)
- moved C2 0.41 mm to (51.5, 26.2)
Routing:
- net /3V3: track 176.2 -> 184.7 mm
- net /BUS_SDA: track 86.6 -> 89.1 mm
- net /BUS_SCL: track 101.3 -> 102.9 mm
