File: LCD320x240/KiCAD/BarePi_LCD320x240.kicad_pcb (KiCad board)
At the start: 2 copper layers, 65 x 49 mm, 16 parts, among them J1 IN, J2 OUT, J3 LCD, J4 WCH-LINK, U1 CH32V002J4M6

Commit message: init
Parts:
- added R2: 15K, Resistor_SMD:R_1206_3216Metric_Pad1.30x1.75mm_HandSolder, B.Cu at (15.4, 13.7)
- added R3: 15K, Resistor_SMD:R_1206_3216Metric_Pad1.30x1.75mm_HandSolder, B.Cu at (12.8, 11.1)
- R1: value 10K -> 15K
Routing:
- net /5V: track 43.7 -> 44.3 mm
