File: LCD320x240/KiCAD/BarePi_LCD320x240.kicad_sch (KiCad schematic)
At the start: 12 parts, among them J1 IN, J2 OUT, J3 LCD, J4 WCH-LINK, U1 CH32V002J4M6

Commit message: init
Parts:
- added R2, R3: 15K, Resistor_SMD:R_1206_3216Metric_Pad1.30x1.75mm_HandSolder, symbol Device:R
- R1: value 10K -> 15K
Connections:
- net 3V3: now also R2.2, R3.2
- net BUS_SCL: now also R3.1
- net BUS_SDA: now also R2.1
Other:
- moved on the sheet: C2, J4, JP1, JP2, U1
