File: LED12/KiCAD/BarePi_LED12.kicad_pcb (KiCad board)
At the start: 2 copper layers, 90 x 50 mm, 21 parts, among them J1 IN, J2 OUT, J3 WCH-LINK, U1 CH32V006E8R6

Commit message: init
Parts:
- added R10: 15K, Resistor_SMD:R_1206_3216Metric_Pad1.30x1.75mm_HandSolder, B.Cu at (32.8, 30.0)
- added R9: 15K, Resistor_SMD:R_1206_3216Metric_Pad1.30x1.75mm_HandSolder, B.Cu at (29.4, 30.0)
Routing:
- net /BUS_SCL: track 58.1 -> 66.9 mm
- net /BUS_SDA: track 61.1 -> 64.7 mm, vias 2 -> 3
- net /3V3: track 130.7 -> 131.7 mm
- net /SWIO: track 85.0 -> 84.5 mm
