File: MegaTinyJoypad/KiCAD/BarePi_MegaTinyJoypad.kicad_pcb (KiCad board)
At the start: 2 copper layers, 65 x 38 mm, 9 parts, among them J1 OUT, J2 L, J3 R, U2 ESP-07S

Commit message: init
Parts:
- added R1: 15K, Resistor_SMD:R_1206_3216Metric_Pad1.30x1.75mm_HandSolder, B.Cu at (33.3, 13.0)
- added R2: 15K, Resistor_SMD:R_1206_3216Metric_Pad1.30x1.75mm_HandSolder, B.Cu at (33.3, 8.80)
Routing:
- net /3V3: track 24.5 -> 38.0 mm
- net /I2C_SCL: track 45.5 -> 48.3 mm
- net /I2C_SDA: track 47.5 -> 48.9 mm
