File: MiniKey/KiCAD/BarePi_MiniKey.kicad_pcb (KiCad board)
At the start: 2 copper layers, 100 x 75 mm, 59 parts, among them J1 IN, J2 WCH-LINK, SW1 1 ! F1, SW10 0 ) F10, SW11 Q \ Query, SW12 W | Close, SW13 E ` Move, SW14 R ~ Replace, SW15 T < Ins, SW16 Y > Redo, SW17 U = Home, SW18 I / Tab, SW19 O + Open, SW2 2 @ F2, SW20 P - Print, SW21 A Vol- All, SW22 S Vol+ Save, SW23 D _ End, SW24 F [ Find, SW25 G ] Next, SW26 H ; Back, SW27 J : Line, SW28 K " PgUp, SW29 L ' PgDn, SW3 3 # F3, SW30 BS Del, SW31 Z Disp- Undo, SW32 X Disp+ Cut, SW33 C { Copy, SW34 V } Paste, SW35 B , Block, SW36 N . New, SW37 M ? Enter, SW38 Up PgUp, SW39 Enter Edit [B], SW4 4 $ F4, SW40 Alt, SW41 Shift Caps, SW42 Ctrl, SW43 Space Ins Nul [A], SW44 Tab PrtScr [X], SW45 Esc Menu Break [Y], SW46 Left Home, SW47 Down PgDn, SW48 Right End, SW5 5 % F5, SW6 6 ^ F6, SW7 7 & F7, SW8 8 * F8, SW9 9 ( F9, U1 CH32V002F4P6

Commit message: init
Parts:
- added R2: 15K, Resistor_SMD:R_1206_3216Metric_Pad1.30x1.75mm_HandSolder, B.Cu at (25.2, 13.6)
- added R3: 15K, Resistor_SMD:R_1206_3216Metric_Pad1.30x1.75mm_HandSolder, B.Cu at (25.2, 11.0)
- SW39: value Enter Edit [B] -> Enter Ins [B]
- SW43: value Space Ins Nul [A] -> Space Zoom Nul [A]
Routing:
- net /BUS_SDA: track 19.4 -> 25.2 mm
- net /3V3: track 86.7 -> 91.0 mm
- net /BUS_SCL: track 21.1 -> 23.6 mm
