File: MiniKey/KiCAD/BarePi_MiniKey.kicad_sch (KiCad schematic)
At the start: 55 parts, among them J1 IN, J2 WCH-LINK, SW1 1 ! F1, SW10 0 ) F10, SW11 Q \ Query, SW12 W | Close, SW13 E ` Move, SW14 R ~ Replace, SW15 T < Ins, SW16 Y > Redo, SW17 U = Home, SW18 I / Tab, SW19 O + Open, SW2 2 @ F2, SW20 P - Print, SW21 A Vol- All, SW22 S Vol+ Save, SW23 D _ End, SW24 F [ Find, SW25 G ] Next, SW26 H ; Back, SW27 J : Line, SW28 K {dblquote} PgUp, SW29 L ' PgDn, SW3 3 # F3, SW30 BS Del, SW31 Z Disp- Undo, SW32 X Disp+ Cut, SW33 C { Copy, SW34 V } Paste, SW35 B , Block, SW36 N . New, SW37 M ? Enter, SW38 Up PgUp, SW39 Enter Edit [B], SW4 4 $ F4, SW40 Alt, SW41 Shift Caps, SW42 Ctrl, SW43 Space Ins Nul [A], SW44 Tab PrtScr [X], SW45 Esc Menu Break [Y], SW46 Left Home, SW47 Down PgDn, SW48 Right End, SW5 5 % F5, SW6 6 ^ F6, SW7 7 & F7, SW8 8 * F8, SW9 9 ( F9, U1 CH32V002F4P6

Commit message: init
Parts:
- added R2, R3: 15K, Resistor_SMD:R_1206_3216Metric_Pad1.30x1.75mm_HandSolder, symbol Device:R
- SW39: value Enter Edit [B] -> Enter Ins [B]
- SW43: value Space Ins Nul [A] -> Space Zoom Nul [A]
Connections:
- net 3V3: now also R2.2, R3.2
- net BUS_SCL: now also R3.1
- net BUS_SDA: now also R2.1
Other:
- moved on the sheet: C1
Changed lines of the file:
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@@
 	)
 	(junction
+		(at 152.4 22.86)
+		(diameter 0)
+		(color 0 0 0 0)
+	)
+	(junction
 		(at 210.82 91.44)
 		(diameter 0)
@@
 	(wire
 		(pts
-			(xy 154.94 38.1) (xy 165.1 38.1)
-		)
-		(stroke
-			(width 0)
-			(type default)
-		)
-	)
-	(wire
-		(pts
 			(xy 111.76 25.4) (xy 124.46 25.4)
 		)
@@
 	(wire
 		(pts
+			(xy 144.78 22.86) (xy 144.78 25.4)
+		)
+		(stroke
+			(width 0)
+			(type default)
+		)
+	)
+	(wire
+		(pts
 			(xy 111.76 121.92) (xy 129.54 121.92)
 		)
@@
 	(wire
 		(pts
-			(xy 139.7 40.64) (xy 139.7 48.26)
+			(xy 132.08 40.64) (xy 132.08 48.26)
 		)
 		(stroke
@@
 	(wire
 		(pts
-			(xy 139.7 30.48) (xy 139.7 35.56)
+			(xy 132.08 30.48) (xy 132.08 35.56)
 		)
 		(stroke
@@
 	(wire
 		(pts
+			(xy 152.4 22.86) (xy 144.78 22.86)
+		)
+		(stroke
+			(width 0)
+			(type default)
+		)
+	)
+	(wire
+		(pts
 			(xy 93.98 121.92) (xy 111.76 121.92)
 		)
@@
 	(wire
 		(pts
+			(xy 154.94 22.86) (xy 152.4 22.86)
+		)
+		(stroke
+			(width 0)
+			(type default)
+		)
+	)
+	(wire
+		(pts
 			(xy 63.5 25.4) (xy 76.2 25.4)
 		)
@@
 	(wire
 		(pts
+			(xy 144.78 38.1) (xy 165.1 38.1)
+		)
+		(stroke
+			(width 0)
+			(type default)
+		)
+	)
+	(wire
+		(pts
 			(xy 185.42 55.88) (xy 190.5 55.88)
 		)
@@
 	(wire
 		(pts
+			(xy 152.4 22.86) (xy 152.4 25.4)
+		)
+		(stroke
+			(width 0)
+			(type default)
+		)
+	)
+	(wire
+		(pts
 			(xy 228.6 134.62) (xy 228.6 149.86)
 		)
@@
 	(wire
 		(pts
+			(xy 144.78 33.02) (xy 144.78 38.1)
+		)
+		(stroke
+			(width 0)
+			(type default)
+		)
+	)
+	(wire
+		(pts
 			(xy 205.74 134.62) (xy 205.74 149.86)
 		)
@@
 	(wire
 		(pts
-			(xy 154.94 35.56) (xy 165.1 35.56)
-		)
-		(stroke
-			(width 0)
-			(type default)
-		)
-	)
-	(wire
-		(pts
 			(xy 172.72 149.86) (xy 172.72 154.94)
 		)
@@
 	(wire
 		(pts
+			(xy 152.4 33.02) (xy 152.4 35.56)
+		)
+		(stroke
+			(width 0)
+			(type default)
+		)
+	)
+	(wire
+		(pts
 			(xy 175.26 91.44) (xy 193.04 91.44)
 		)
@@
 	(wire
 		(pts
+			(xy 152.4 35.56) (xy 165.1 35.56)
+		)
+		(stroke
+			(width 0)
+			(type default)
+		)
+	)
+	(wire
+		(pts
 			(xy 139.7 119.38) (xy 147.32 119.38)
 		)
@@
 	)
 	(label "3V3"
-		(at 139.7 30.48 0)
+		(at 132.08 30.48 0)
 		(effects
 			(font
@@
 	)
 	(label "GND"
-		(at 139.7 48.26 0)
+		(at 132.08 48.26 0)
 		(effects
 			(font
@@
 		)
 	)
+	(label "3V3"
+		(at 154.94 22.86 0)
+		(effects
+			(font
+				(size 1.27 1.27)
+			)
+			(justify left bottom)
+		)
+	)
 	(label "GND"
 		(at 144.78 154.94 0)
@@
 	)
 	(symbol
+		(lib_id "Device:R")
+		(at 152.4 29.21 180)
+		(unit 1)
+		(exclude_from_sim no)
+		(in_bom yes)
+		(on_board yes)
+		(dnp no)
+		(property "Reference" "R2"
+			(at 149.225 30.48 0)
+			(effects
+				(font
+					(size 1.27 1.27)
+				)
+			)
+		)
+		(property "Value" "15K"
+			(at 149.225 27.305 0)
+			(effects
+				(font
+					(size 1.27 1.27)
+				)
+			)
+		)
+		(property "Footprint" "Resistor_SMD:R_1206_3216Metric_Pad1.30x1.75mm_HandSolder"
+			(at 154.178 29.21 90)
+			(effects
+				(font
+					(size 1.27 1.27)
+				)
+				(hide yes)
+			)
+		)
+		(property "Datasheet" "~"
+			(at 152.4 29.21 0)
+			(effects
+				(font
+					(size 1.27 1.27)
+				)
+				(hide yes)
+			)
+		)
+		(property "Description" "Resistor"
+			(at 152.4 29.21 0)
+			(effects
+				(font
+					(size 1.27 1.27)
+				)
+				(hide yes)
+			)
+		)
+		(pin "2"
+		)
+		(pin "1"
+		)
+		(instances
+			(project "BarePi_MiniKey"
+				(path "/b3c66170-a1e8-49f2-a3c7-446e9ba3066c"
+					(reference "R2")
+					(unit 1)
+				)
+			)
+		)
+	)
+	(symbol
 		(lib_id "Jumper:SolderJumper_2_Bridged")
 		(at 194.31 55.88 0)
@@
 			)
 		)
-		(property "Value" "Enter Edit [B]"
+		(property "Value" "Enter Ins [B]"
 			(at 223.52 129.54 0)
 			(effects
@@
 	(symbol
 		(lib_id "Device:C_Small")
-		(at 139.7 38.1 0)
+		(at 132.08 38.1 0)
 		(unit 1)
 		(exclude_from_sim no)
@@
 		(fields_autoplaced yes)
 		(property "Reference" "C1"
-			(at 142.24 36.8362 0)
+			(at 134.62 36.8362 0)
 			(effects
 				(font
@@
 		)
 		(property "Value" "100nF"
-			(at 142.24 39.3762 0)
+			(at 134.62 39.3762 0)
 			(effects
 				(font
@@
 		)
 		(property "Footprint" "Capacitor_SMD:C_1210_3225Metric_Pad1.33x2.70mm_HandSolder"
-			(at 139.7 38.1 0)
+			(at 132.08 38.1 0)
 			(effects
 				(font
@@
 		)
 		(property "Datasheet" "~"
-			(at 139.7 38.1 0)
+			(at 132.08 38.1 0)
 			(effects
 				(font
@@
 		)
 		(property "Description" "Unpolarized capacitor, small symbol"
-			(at 139.7 38.1 0)
+			(at 132.08 38.1 0)
 			(effects
 				(font
@@
 	)
 	(symbol
+		(lib_id "Device:R")
+		(at 144.78 29.21 180)
+		(unit 1)
+		(exclude_from_sim no)
+		(in_bom yes)
+		(on_board yes)
+		(dnp no)
+		(property "Reference" "R3"
+			(at 142.24 30.48 0)
+			(effects
+				(font
+					(size 1.27 1.27)
+				)
+			)
+		)
+		(property "Value" "15K"
+			(at 141.605 27.305 0)
+			(effects
+				(font
+					(size 1.27 1.27)
+				)
+			)
+		)
+		(property "Footprint" "Resistor_SMD:R_1206_3216Metric_Pad1.30x1.75mm_HandSolder"
+			(at 146.558 29.21 90)
+			(effects
+				(font
+					(size 1.27 1.27)
+				)
+				(hide yes)
+			)
+		)
+		(property "Datasheet" "~"
+			(at 144.78 29.21 0)
+			(effects
+				(font
+					(size 1.27 1.27)
+				)
+				(hide yes)
+			)
+		)
+		(property "Description" "Resistor"
+			(at 144.78 29.21 0)
+			(effects
+				(font
+					(size 1.27 1.27)
+				)
+				(hide yes)
+			)
+		)
+		(pin "2"
+		)
+		(pin "1"
+		)
+		(instances
+			(project "BarePi_MiniKey"
+				(path "/b3c66170-a1e8-49f2-a3c7-446e9ba3066c"
+					(reference "R3")
+					(unit 1)
+				)
+			)
+		)
+	)
+	(symbol
 		(lib_id "Switch:SW_Push")
 		(at 99.06 149.86 0)
@@
 			)
 		)
-		(property "Value" "Space Ins Nul [A]"
+		(property "Value" "Space Zoom Nul [A]"
 			(at 119.38 144.78 0)
 			(effects
