File: PGA2350/KiCAD/BarePi_PGA2350.kicad_pcb (KiCad board)
At the start: 2 copper layers, 65 x 65 mm, 19 parts, among them J1 OUT, J2 DISPLAY, J3 USB, SW1 BOOTSEL, U1 PGA2350

Commit message: init
Parts:
- added R10: 15K, Resistor_SMD:R_1206_3216Metric_Pad1.30x1.75mm_HandSolder, F.Cu at (14.0, 47.8)
- added R7: 15K, Resistor_SMD:R_1206_3216Metric_Pad1.30x1.75mm_HandSolder, F.Cu at (11.9, 37.0)
- added R8: 15K, Resistor_SMD:R_1206_3216Metric_Pad1.30x1.75mm_HandSolder, F.Cu at (14.6, 43.0)
- added R9: 15K, Resistor_SMD:R_1206_3216Metric_Pad1.30x1.75mm_HandSolder, F.Cu at (13.2, 40.2)
Routing:
- net /GND: track 363.6 -> 353.6 mm
- net /3V3: track 90.6 -> 99.6 mm
- net /BUS_SDA: track 38.2 -> 42.5 mm
- net /I2C_SDA: track 40.9 -> 44.8 mm
- net /I2C_SCL: track 36.4 -> 39.1 mm
- net /USB_DP: track 82.7 -> 84.7 mm
- net /BUS_SCL: track 36.9 -> 38.7 mm
- net /USB_DM: track 77.8 -> 79.3 mm
