File: PicoPad/KiCAD/BarePi_PicoPad.kicad_pcb (KiCad board)
At the start: 2 copper layers, 65 x 45 mm, 6 parts, among them IC1 Raspberry Pi Pico, J1 OUT

Commit message: init
Parts:
- added R1: 15K, Resistor_SMD:R_1206_3216Metric_Pad1.30x1.75mm_HandSolder, B.Cu at (9.12, 28.5)
- added R2: 15K, Resistor_SMD:R_1206_3216Metric_Pad1.30x1.75mm_HandSolder, B.Cu at (9.12, 24.7)
Routing:
- net /3V3: track 61.5 -> 72.1 mm
- net /I2C_SCL: track 62.8 -> 72.6 mm
- net /I2C_SDA: track 43.6 -> 52.2 mm
