File: PidiBoy/KiCAD/BarePi_PidiBoy.kicad_pcb (KiCad board)
At the start: 2 copper layers, 65 x 26 mm, 8 parts, among them IC1 CH32V006F8P6, J1 OUT, J2 WCH-LINK

Commit message: init
Parts:
- added R1: 15K, Resistor_SMD:R_1206_3216Metric_Pad1.30x1.75mm_HandSolder, F.Cu at (11.4, 9.44)
- added R2: 15K, Resistor_SMD:R_1206_3216Metric_Pad1.30x1.75mm_HandSolder, F.Cu at (12.6, 5.66)
Routing:
- net /3V3: track 76.6 -> 86.2 mm
- net /I2C_SCL: track 28.5 -> 37.9 mm
- net /I2C_SDA: track 26.0 -> 34.7 mm
