File: Port/KiCAD/BarePi_Port.kicad_pcb (KiCad board)
At the start: 2 copper layers, 65 x 65 mm, 18 parts, among them J1 IN, J10 SPI1, J11 PORT, J12 UART, J2 OUT, J3 WCH-LINK, J4 I2C, J5 I2C, J6 I2C, J7 SPI0, J8 SPI1, J9 SPI0, U1 CH32V002A4M6

Commit message: init
Parts:
- added R1: 15K, Resistor_SMD:R_1206_3216Metric_Pad1.30x1.75mm_HandSolder, F.Cu at (5.21, 45.5)
- added R2: 15K, Resistor_SMD:R_1206_3216Metric_Pad1.30x1.75mm_HandSolder, F.Cu at (4.63, 49.2)
Routing:
- net /3V3: track 191.9 -> 198.9 mm
- net /BUS_SCL: track 83.1 -> 89.4 mm
- net /BUS_SDA: track 92.9 -> 98.3 mm
