File: RTC/KiCAD/BarePi_RTC.kicad_pcb (KiCad board)
At the start: 2 copper layers, 65 x 48 mm, 15 parts, among them J1 IN, J2 OUT, J3 EEPROM1, J4 EEPROM2, U1 DS3231, U2 AT24C32

Commit message: init
Parts:
- R1: renamed from R2; value 10K -> 15K
- R2: renamed from R1; value 10K -> 15K
Changed lines of the file:
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@@
 		(descr "Resistor SMD 1206 (3216 Metric), square (rectangular) end terminal, IPC-7351 nominal with elongated pad for handsoldering. (Body size source: IPC-SM-782 page 72, https://www.pcb-3d.com/wordpress/wp-content/uploads/ipc-sm-782a_amendment_1_and_2.pdf), generated with kicad-footprint-generator")
 		(tags "resistor handsolder")
-		(property "Reference" "R1"
+		(property "Reference" "R2"
 			(at 3.08 -0.54 0)
 			(layer "F.SilkS")
@@
 			)
 		)
-		(property "Value" "10K"
+		(property "Value" "15K"
 			(at 2.73 1.8 0)
 			(layer "F.Fab")
@@
 		(descr "Resistor SMD 1206 (3216 Metric), square (rectangular) end terminal, IPC-7351 nominal with elongated pad for handsoldering. (Body size source: IPC-SM-782 page 72, https://www.pcb-3d.com/wordpress/wp-content/uploads/ipc-sm-782a_amendment_1_and_2.pdf), generated with kicad-footprint-generator")
 		(tags "resistor handsolder")
-		(property "Reference" "R2"
+		(property "Reference" "R1"
 			(at 0.76 -1.91 0)
 			(layer "F.SilkS")
@@
 			)
 		)
-		(property "Value" "10K"
+		(property "Value" "15K"
 			(at 3.82 -1.27 0)
 			(layer "F.Fab")
