File: RTC/KiCAD/BarePi_RTC.kicad_sch (KiCad schematic)
At the start: 11 parts, among them J1 IN, J2 OUT, J3 EEPROM1, J4 EEPROM2, U1 DS3231, U2 AT24C32

Commit message: init
Parts:
- R1: renamed from R2; value 10K -> 15K
- R2: renamed from R1; value 10K -> 15K
Changed lines of the file:
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@@
 		(on_board yes)
 		(dnp no)
-		(property "Reference" "R1"
+		(property "Reference" "R2"
 			(at 120.015 116.2049 0)
 			(effects
@@
 			)
 		)
-		(property "Value" "10K"
+		(property "Value" "15K"
 			(at 118.745 118.7449 0)
 			(effects
@@
 			(project ""
 				(path "/b3c66170-a1e8-49f2-a3c7-446e9ba3066c"
-					(reference "R1")
+					(reference "R2")
 					(unit 1)
 				)
@@
 		(on_board yes)
 		(dnp no)
-		(property "Reference" "R2"
+		(property "Reference" "R1"
 			(at 131.445 116.2049 0)
 			(effects
@@
 			)
 		)
-		(property "Value" "10K"
+		(property "Value" "15K"
 			(at 131.445 118.7449 0)
 			(effects
@@
 			(project "BarePi_RTC"
 				(path "/b3c66170-a1e8-49f2-a3c7-446e9ba3066c"
-					(reference "R2")
-					(unit 1)
-				)
+					(reference "R1")
+					(unit 1)
+				)
