File: SumoPad/KiCAD/BarePi_SumoPad.kicad_pcb (KiCad board)
At the start: 2 copper layers, 65 x 65 mm, 21 parts, among them J1 OUT, J2 WCH-LINK, J3 DISPLAY, J4 USB, Q1 24MHz, U1 CH32V208RBT6

Commit message: init
Parts:
- added R10: 15K, Resistor_SMD:R_1206_3216Metric_Pad1.30x1.75mm_HandSolder, F.Cu at (17.9, 37.1)
- added R11: 15K, Resistor_SMD:R_1206_3216Metric_Pad1.30x1.75mm_HandSolder, F.Cu at (15.0, 46.4)
- added R12: 15K, Resistor_SMD:R_1206_3216Metric_Pad1.30x1.75mm_HandSolder, F.Cu at (20.5, 35.8)
- added R9: 15K, Resistor_SMD:R_1206_3216Metric_Pad1.30x1.75mm_HandSolder, F.Cu at (14.9, 42.1)
Routing:
- net /3V3: track 145.3 -> 168.3 mm
- net /I2C_SDA: track 76.6 -> 87.5 mm
- net /BUS_SCL: track 54.7 -> 57.1 mm
- net /BUS_SDA: track 51.4 -> 52.9 mm
