File: SumoPad/KiCAD/BarePi_SumoPad.kicad_sch (KiCad schematic)
At the start: 17 parts, among them J1 OUT, J2 WCH-LINK, J3 DISPLAY, J4 USB, Q1 24MHz, U1 CH32V208RBT6

Commit message: init
Parts:
- added R10, R11, R12, R9: 15K, Resistor_SMD:R_1206_3216Metric_Pad1.30x1.75mm_HandSolder, symbol Device:R
Connections:
- net 3V3: now also R10.1, R11.1, R12.1, R9.1
- net BUS_SCL: now also R10.2
- net BUS_SDA: now also R9.2
- net I2C_SCL: now also R12.2
- net I2C_SDA: now also R11.2
Other:
- moved on the sheet: J3, R1, R2, R3, R4, R5, R6
