File: TweetyBoy/KiCAD/BarePi_TweetyBoy.kicad_pcb (KiCad board)
At the start: 2 copper layers, 65 x 28 mm, 8 parts, among them IC1 CH32X035G8R6, J1 OUT, J2 WCH-LINK

Commit message: init
Parts:
- added R1: 15K, Resistor_SMD:R_1206_3216Metric_Pad1.30x1.75mm_HandSolder, B.Cu at (12.9, 6.62)
- added R2: 15K, Resistor_SMD:R_1206_3216Metric_Pad1.30x1.75mm_HandSolder, B.Cu at (12.9, 9.56)
Routing:
- net /3V3: track 71.4 -> 76.9 mm
- net /GND: track 154.6 -> 157.8 mm
- net /I2C_SDA: track 34.3 -> 36.5 mm
- net /I2C_SCL: track 32.8 -> 34.7 mm
