File: Zero/KiCAD/BarePi_Zero.kicad_pcb (KiCad board)
At the start: 2 copper layers, 65 x 48 mm, 4 parts, among them J1 Raspberry_Pi_Zero, J2 OUT

Commit message: init
Parts:
- added R1: 15K, Resistor_SMD:R_1206_3216Metric_Pad1.30x1.75mm_HandSolder, B.Cu at (12.4, 12.8)
- added R2: 15K, Resistor_SMD:R_1206_3216Metric_Pad1.30x1.75mm_HandSolder, B.Cu at (5.38, 12.8)
- added R3: 15K, Resistor_SMD:R_1206_3216Metric_Pad1.30x1.75mm_HandSolder, B.Cu at (8.88, 12.8)
- added R4: 15K, Resistor_SMD:R_1206_3216Metric_Pad1.30x1.75mm_HandSolder, B.Cu at (15.9, 12.8)
Routing:
- net /3V3: track 59.5 -> 84.8 mm
- net /BUS_SCL: track 41.5 -> 64.2 mm, vias 2 -> 3
- net /I2C_SCL: track 12.2 -> 24.1 mm
- net /I2C_SDA: track 27.5 -> 36.4 mm
- net /BUS_SDA: track 59.5 -> 65.1 mm
